File: canGaugeDriver.kicad_sch (KiCad schematic)
At the start: 35 parts, among them J1 CANbed 1.0 Interface, J2 VIN INTERFACE, J3 BLUESMIRF, J4 1848710, U1 TPL7407LA, U2 TPL7407LA

Commit message: fixed headers
Parts:
- removed J3: BLUESMIRF, Connector_PinHeader_2.54mm:PinHeader_1x06_P2.54mm_Vertical, symbol Connector_Generic:Conn_01x06
- J1: symbol Connector_Generic:Conn_02x09_Top_Bottom -> Connector_Generic:Conn_02x09_Odd_Even
Connections:
- net 5V: now also J1.17 (Pin_17); no longer J1.9 (Pin_9)
- net A0: now also J1.11 (Pin_11); no longer J1.6 (Pin_6)
- net A1: now also J1.13 (Pin_13); no longer J1.7 (Pin_7)
- net A2: now also J1.15 (Pin_15); no longer J1.8 (Pin_8)
- net A3: now also J1.7 (Pin_7); no longer J1.4 (Pin_4)
- net D0_RX: now also J1.2 (Pin_2); no longer J1.10 (Pin_10)
- net D10_OIL: now also J1.14 (Pin_14); no longer J1.16 (Pin_16)
- net D11_TACH: now also J1.16 (Pin_16); no longer J1.17 (Pin_17)
- net D12_ALT: now also J1.9 (Pin_9); no longer J1.5 (Pin_5)
- net D1_TX: now also J1.4 (Pin_4); no longer J1.11 (Pin_11)
- net D2_SRS: now also J1.6 (Pin_6); no longer J1.12 (Pin_12)
- net D3_SPEED: now also J1.8 (Pin_8); no longer J1.13 (Pin_13)
- net D5_COOL: now also J1.3 (Pin_3); no longer J1.2 (Pin_2)
- net D6_ABS: now also J1.5 (Pin_5); no longer J1.3 (Pin_3)
- net D8_SEATBELT: now also J1.10 (Pin_10); no longer J1.14 (Pin_14)
- net D9_FUEL: now also J1.12 (Pin_12); no longer J1.15 (Pin_15)
Changed lines of the file:
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@@
 	(wire
 		(pts
-			(xy 232.41 54.61) (xy 248.92 54.61)
-		)
-		(stroke
-			(width 0)
-			(type default)
-		)
-	)
-	(wire
-		(pts
 			(xy 161.29 62.23) (xy 171.45 62.23)
 		)
@@
 	(wire
 		(pts
-			(xy 245.11 63.5) (xy 245.11 62.23)
-		)
-		(stroke
-			(width 0)
-			(type default)
-		)
-	)
-	(wire
-		(pts
 			(xy 215.9 125.73) (xy 215.9 146.05)
 		)
@@
 	(wire
 		(pts
-			(xy 232.41 52.07) (xy 248.92 52.07)
-		)
-		(stroke
-			(width 0)
-			(type default)
-		)
-	)
-	(wire
-		(pts
 			(xy 193.04 138.43) (xy 226.06 138.43)
 		)
@@
 	(wire
 		(pts
-			(xy 245.11 62.23) (xy 248.92 62.23)
-		)
-		(stroke
-			(width 0)
-			(type default)
-		)
-	)
-	(wire
-		(pts
 			(xy 36.83 134.62) (xy 36.83 133.35)
 		)
@@
 	(wire
 		(pts
-			(xy 232.41 57.15) (xy 248.92 57.15)
-		)
-		(stroke
-			(width 0)
-			(type default)
-		)
-	)
-	(wire
-		(pts
 			(xy 91.44 130.81) (xy 91.44 132.08)
 		)
@@
 		)
 	)
-	(label "5V"
-		(at 232.41 57.15 0)
-		(effects
-			(font
-				(size 1.27 1.27)
-			)
-			(justify left bottom)
-		)
-	)
 	(label "D3_OUT"
 		(at 161.29 64.77 0)
@@
 		)
 	)
-	(label "EXT_SERIAL_RX"
-		(at 232.41 52.07 0)
-		(effects
-			(font
-				(size 1.27 1.27)
-			)
-			(justify left bottom)
-		)
-	)
 	(label "A2"
 		(at 30.48 55.88 0)
@@
 		)
 	)
-	(label "EXT_SERIAL_TX"
-		(at 232.41 54.61 0)
-		(effects
-			(font
-				(size 1.27 1.27)
-			)
-			(justify left bottom)
-		)
-	)
 	(label "D3_SPEED"
 		(at 140.97 133.35 0)
@@
 	)
 	(symbol
-		(lib_id "Connector_Generic:Conn_02x09_Top_Bottom")
+		(lib_id "Connector_Generic:Conn_02x09_Odd_Even")
 		(at 45.72 48.26 0)
 		(unit 1)
@@
 			)
 		)
-		(property "Description" "Generic connector, double row, 02x09, top/bottom pin numbering scheme (row 1: 1...pins_per_row, row2: pins_per_row+1 ... num_pins), script generated (kicad-library-utils/schlib/autogen/connector/)"
+		(property "Description" "Generic connector, double row, 02x09, odd/even pin numbering scheme (row 1 odd numbers, row 2 even numbers), script generated (kicad-library-utils/schlib/autogen/connector/)"
 			(at 45.72 48.26 0)
 			(hide yes)
@@
 	)
 	(symbol
-		(lib_id "Connector_Generic:Conn_01x06")
-		(at 254 54.61 0)
-		(unit 1)
-		(body_style 1)
-		(exclude_from_sim no)
-		(in_bom yes)
-		(on_board yes)
-		(in_pos_files yes)
-		(dnp no)
-		(fields_autoplaced yes)
-		(property "Reference" "J3"
-			(at 256.54 54.6099 0)
-			(show_name no)
-			(do_not_autoplace no)
-			(effects
-				(font
-					(size 1.27 1.27)
-				)
-				(justify left)
-			)
-		)
-		(property "Value" "BLUESMIRF"
-			(at 256.54 57.1499 0)
-			(show_name no)
-			(do_not_autoplace no)
-			(effects
-				(font
-					(size 1.27 1.27)
-				)
-				(justify left)
-			)
-		)
-		(property "Footprint" "Connector_PinHeader_2.54mm:PinHeader_1x06_P2.54mm_Vertical"
-			(at 254 54.61 0)
-			(hide yes)
-			(show_name no)
-			(do_not_autoplace no)
-			(effects
-				(font
-					(size 1.27 1.27)
-				)
-			)
-		)
-		(property "Datasheet" ""
-			(at 254 54.61 0)
-			(hide yes)
-			(show_name no)
-			(do_not_autoplace no)
-			(effects
-				(font
-					(size 1.27 1.27)
-				)
-			)
-		)
-		(property "Description" "Generic connector, single row, 01x06, script generated (kicad-library-utils/schlib/autogen/connector/)"
-			(at 254 54.61 0)
-			(hide yes)
-			(show_name no)
-			(do_not_autoplace no)
-			(effects
-				(font
-					(size 1.27 1.27)
-				)
-			)
-		)
-		(pin "3"
-		)
-		(pin "2"
-		)
-		(pin "6"
-		)
-		(pin "4"
-		)
-		(pin "5"
-		)
-		(pin "1"
-		)
-		(instances
-			(project "canGaugeDriver"
-				(path "/53705195-86fb-46bf-a563-00a6cdeeae38"
-					(reference "J3")
-					(unit 1)
-				)
-			)
-		)
-	)
-	(symbol
 		(lib_id "1848710:1848710")
 		(at 184.15 57.15 0)
@@
 					(unit 1)
 				)
-			)
-		)
-	)
-	(symbol
-		(lib_id "power:GND")
-		(at 245.11 63.5 0)
-		(unit 1)
-		(body_style 1)
-		(exclude_from_sim no)
-		(in_bom yes)
-		(on_board yes)
-		(in_pos_files yes)
-		(dnp no)
-		(fields_autoplaced yes)
-		(property "Reference" "#PWR02"
-			(at 245.11 69.85 0)
-			(hide yes)
-			(show_name no)
-			(do_not_autoplace no)
-			(effects
-				(font
-					(size 1.27 1.27)
-				)
-			)
-		)
-		(property "Value" "GND"
-			(at 245.11 68.58 0)
-			(show_name no)
-			(do_not_autoplace no)
-			(effects
-				(font
-					(size 1.27 1.27)
-				)
-			)
-		)
-		(property "Footprint" ""
-			(at 245.11 63.5 0)
-			(hide yes)
-			(show_name no)
-			(do_not_autoplace no)
-			(effects
-				(font
-					(size 1.27 1.27)
-				)
-			)
-		)
-		(property "Datasheet" ""
-			(at 245.11 63.5 0)
-			(hide yes)
-			(show_name no)
-			(do_not_autoplace no)
-			(effects
-				(font
-					(size 1.27 1.27)
-				)
-			)
-		)
-		(property "Description" "Power symbol creates a global label with name \"GND\" , ground"
-			(at 245.11 63.5 0)
-			(hide yes)
-			(show_name no)
-			(do_not_autoplace no)
-			(effects
-				(font
-					(size 1.27 1.27)
-				)
-			)
-		)
-		(pin "1"
-		)
-		(instances
-			(project "canGaugeDriver"
-				(path "/53705195-86fb-46bf-a563-00a6cdeeae38"
-					(reference "#PWR02")
-					(unit 1)
-				)

Commit message: replaced output connector
Parts:
- removed J4: 1848710, PHOENIX_1848710:PHOENIX_1848710, symbol 1848710:1848710
- added J3: 348260240, CONN_SD-34826-001_24_MOL, symbol 348260240:348260240
Changed lines of the file:
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@@
-	)
-	(symbol
-		(lib_id "1848710:1848710")
-		(at 184.15 57.15 0)
-		(unit 1)
-		(body_style 1)
-		(exclude_from_sim no)
-		(in_bom yes)
-		(on_board yes)
-		(in_pos_files yes)
-		(dnp no)
-		(fields_autoplaced yes)
-		(property "Reference" "J4"
-			(at 184.15 39.37 0)
-			(show_name no)
-			(do_not_autoplace no)
-			(effects
-				(font
-					(size 1.27 1.27)
-				)
-			)
-		)
-		(property "Value" "1848710"
-			(at 184.15 41.91 0)
-			(show_name no)
-			(do_not_autoplace no)
-			(effects
-				(font
-					(size 1.27 1.27)
-				)
-			)
-		)
-		(property "Footprint" "PHOENIX_1848710:PHOENIX_1848710"
-			(at 184.15 57.15 0)
-			(hide yes)
-			(show_name no)
-			(do_not_autoplace no)
-			(effects
-				(font
-					(size 1.27 1.27)
-				)
-				(justify bottom)
-			)
-		)
-		(property "Datasheet" "file://Z:\\My Drive\\fastboi\\canGaugeDriver\\datasheets\\1848710_Ds.pdf"
-			(at 184.15 57.15 0)
-			(hide yes)
-			(show_name no)
-			(do_not_autoplace no)
-			(effects
-				(font
-					(size 1.27 1.27)
-				)
-			)
-		)
-		(property "Description" ""
-			(at 184.15 57.15 0)
-			(hide yes)
-			(show_name no)
-			(do_not_autoplace no)
-			(effects
-				(font
-					(size 1.27 1.27)
-				)
-			)
-		)
-		(property "PARTREV" "11.07.2018"
-			(at 184.15 57.15 0)
-			(hide yes)
-			(show_name no)
-			(do_not_autoplace no)
-			(effects
-				(font
-					(size 1.27 1.27)
-				)
-				(justify bottom)
-			)
-		)
-		(property "STANDARD" "Manufacturer Recommendations"
-			(at 184.15 57.15 0)
-			(hide yes)
-			(show_name no)
-			(do_not_autoplace no)
-			(effects
-				(font
-					(size 1.27 1.27)
-				)
-				(justify bottom)
-			)
-		)
-		(property "MAXIMUM_PACKAGE_HEIGHT" "14.15mm"
-			(at 184.15 57.15 0)
-			(hide yes)
-			(show_name no)
-			(do_not_autoplace no)
-			(effects
-				(font
-					(size 1.27 1.27)
-				)
-				(justify bottom)
-			)
-		)
-		(property "MANUFACTURER" "Phoenix Contact"
-			(at 184.15 57.15 0)
-			(hide yes)
-			(show_name no)
-			(do_not_autoplace no)
-			(effects
-				(font
-					(size 1.27 1.27)
-				)
-				(justify bottom)
-			)
-		)
-		(pin "1_8"
-		)
-		(pin "2_5"
-		)
-		(pin "1_6"
-		)
-		(pin "1_5"
-		)
-		(pin "1_1"
-		)
-		(pin "2_3"
-		)
-		(pin "2_4"
-		)
-		(pin "2_7"
-		)
-		(pin "1_7"
-		)
-		(pin "1_4"
-		)
-		(pin "1_2"
-		)
-		(pin "1_3"
-		)
-		(pin "1_9"
-		)
-		(pin "2_1"
-		)
-		(pin "2_2"
-		)
-		(pin "2_8"
-		)
-		(pin "2_9"
-		)
-		(pin "2_6"
-		)
-		(instances
-			(project "canGaugeDriver"
-				(path "/53705195-86fb-46bf-a563-00a6cdeeae38"
-					(reference "J4")
-					(unit 1)
-				)
-			)
-		)
 	)
 	(symbol
@@
 					(unit 1)
 				)
+			)
+		)
+	)
+	(symbol
+		(lib_id "348260240:348260240")
+		(at 228.6 38.1 0)
+		(unit 1)
+		(body_style 1)
+		(exclude_from_sim no)
+		(in_bom yes)
+		(on_board yes)
+		(in_pos_files yes)
+		(dnp no)
+		(fields_autoplaced yes)
+		(property "Reference" "J3"
+			(at 242.57 66.0399 0)
+			(show_name no)
+			(do_not_autoplace no)
+			(effects
+				(font
+					(size 1.524 1.524)
+				)
+				(justify left)
+			)
+		)
+		(property "Value" "348260240"
+			(at 242.57 68.5799 0)
+			(show_name no)
+			(do_not_autoplace no)
+			(effects
+				(font
+					(size 1.524 1.524)
+				)
+				(justify left)
+			)
+		)
+		(property "Footprint" "CONN_SD-34826-001_24_MOL"
+			(at 228.6 38.1 0)
+			(hide yes)
+			(show_name no)
+			(do_not_autoplace no)
+			(effects
+				(font
+					(size 1.27 1.27)
+					(italic yes)
+				)
+			)
+		)
+		(property "Datasheet" "https://www.molex.com/en-us/products/part-detail-pdf/348260240?display=pdf"
+			(at 228.6 38.1 0)
+			(hide yes)
+			(show_name no)
+			(do_not_autoplace no)
+			(effects
+				(font
+					(size 1.27 1.27)
+					(italic yes)
+				)
+			)
+		)
+		(property "Description" ""
+			(at 228.6 38.1 0)
+			(hide yes)
+			(show_name no)
+			(do_not_autoplace no)
+			(effects
+				(font
+					(size 1.27 1.27)
+				)
+			)
+		)
+		(pin "12"
+		)
+		(pin "13"
+		)
+		(pin "14"
+		)
+		(pin "24"
+		)
+		(pin "2"
+		)
+		(pin "5"
+		)
+		(pin "6"
+		)
+		(pin "4"
+		)
+		(pin "3"
+		)
+		(pin "1"
+		)
+		(pin "8"
+		)
+		(pin "19"
+		)
+		(pin "22"
+		)
+		(pin "20"
+		)
+		(pin "10"
+		)
+		(pin "23"
+		)
+		(pin "16"
+		)
+		(pin "21"
+		)
+		(pin "11"
+		)
+		(pin "15"
+		)
+		(pin "9"
+		)
+		(pin "17"
+		)
+		(pin "7"
+		)
+		(pin "18"
+		)
+		(instances
+			(project "canGaugeDriver"
+				(path "/53705195-86fb-46bf-a563-00a6cdeeae38"
+					(reference "J3")
+					(unit 1)
+				)

Commit message: progress
Parts:
- added J4: DB9'MEAL', canGaugeDriver:DB9-MEAL, symbol canGaugeDriver:DB9'MEAL'
- J3: footprint CONN_SD-34826-001_24_MOL -> MOLEX_348260240:CONN_SD-34826-001_24_MOL
Connections:
- net 5V: now also J3.1, J3.2
- net GND: now also J3.11, J3.12, J3.24
- net VIN: now also J3.10
Changed lines of the file:
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@@
 	)
 	(junction
+		(at 224.79 66.04)
+		(diameter 0)
+		(color 0 0 0 0)
+	)
+	(junction
 		(at 193.04 138.43)
 		(diameter 0)
@@
 	)
 	(junction
+		(at 224.79 96.52)
+		(diameter 0)
+		(color 0 0 0 0)
+	)
+	(junction
 		(at 185.42 135.89)
 		(diameter 0)
@@
 	(wire
 		(pts
+			(xy 224.79 96.52) (xy 228.6 96.52)
+		)
+		(stroke
+			(width 0)
+			(type default)
+		)
+	)
+	(wire
+		(pts
 			(xy 38.1 181.61) (xy 38.1 184.15)
 		)
@@
 	(wire
 		(pts
+			(xy 217.17 38.1) (xy 228.6 38.1)
+		)
+		(stroke
+			(width 0)
+			(type default)
+		)
+	)
+	(wire
+		(pts
 			(xy 88.9 161.29) (xy 92.71 161.29)
 		)
@@
 	(wire
 		(pts
+			(xy 228.6 63.5) (xy 224.79 63.5)
+		)
+		(stroke
+			(width 0)
+			(type default)
+		)
+	)
+	(wire
+		(pts
 			(xy 53.34 53.34) (xy 57.15 53.34)
 		)
@@
 	(wire
 		(pts
+			(xy 224.79 96.52) (xy 224.79 97.79)
+		)
+		(stroke
+			(width 0)
+			(type default)
+		)
+	)
+	(wire
+		(pts
 			(xy 36.83 134.62) (xy 36.83 133.35)
 		)
@@
 	(wire
 		(pts
+			(xy 217.17 40.64) (xy 228.6 40.64)
+		)
+		(stroke
+			(width 0)
+			(type default)
+		)
+	)
+	(wire
+		(pts
 			(xy 177.8 115.57) (xy 177.8 118.11)
 		)
@@
 	(wire
 		(pts
+			(xy 224.79 66.04) (xy 224.79 96.52)
+		)
+		(stroke
+			(width 0)
+			(type default)
+		)
+	)
+	(wire
+		(pts
 			(xy 171.45 135.89) (xy 185.42 135.89)
 		)
@@
 	(wire
 		(pts
+			(xy 224.79 66.04) (xy 228.6 66.04)
+		)
+		(stroke
+			(width 0)
+			(type default)
+		)
+	)
+	(wire
+		(pts
 			(xy 259.08 135.89) (xy 271.78 135.89)
 		)
@@
 	(wire
 		(pts
+			(xy 224.79 63.5) (xy 224.79 66.04)
+		)
+		(stroke
+			(width 0)
+			(type default)
+		)
+	)
+	(wire
+		(pts
 			(xy 171.45 130.81) (xy 172.72 130.81)
 		)
@@
 	(wire
 		(pts
+			(xy 217.17 60.96) (xy 228.6 60.96)
+		)
+		(stroke
+			(width 0)
+			(type default)
+		)
+	)
+	(wire
+		(pts
 			(xy 241.3 138.43) (xy 237.49 138.43)
 		)
@@
 		)
 	)
+	(label "5V"
+		(at 217.17 38.1 0)
+		(effects
+			(font
+				(size 1.27 1.27)
+			)
+			(justify left bottom)
+		)
+	)
 	(label "AI1"
 		(at 49.53 161.29 180)
@@
 		)
 	)
+	(label "5V"
+		(at 217.17 40.64 0)
+		(effects
+			(font
+				(size 1.27 1.27)
+			)
+			(justify left bottom)
+		)
+	)
 	(label "A3"
 		(at 30.48 45.72 0)
@@
 		)
 	)
+	(label "VIN"
+		(at 217.17 60.96 0)
+		(effects
+			(font
+				(size 1.27 1.27)
+			)
+			(justify left bottom)
+		)
+	)
 	(label "D4_OUT"
 		(at 161.29 62.23 0)
@@
 	)
 	(symbol
+		(lib_id "canGaugeDriver:DB9'MEAL'")
+		(at 179.07 88.9 0)
+		(unit 1)
+		(body_style 1)
+		(exclude_from_sim no)
+		(in_bom yes)
+		(on_board yes)
+		(in_pos_files yes)
+		(dnp no)
+		(fields_autoplaced yes)
+		(property "Reference" "J4"
+			(at 184.15 88.9 0)
+			(show_name no)
+			(do_not_autoplace no)
+			(effects
+				(font
+					(size 1.778 1.5113)
+				)
+				(justify left)
+			)
+		)
+		(property "Value" "DB9'MEAL'"
+			(at 180.34 93.98 90)
+			(hide yes)
+			(show_name no)
+			(do_not_autoplace no)
+			(effects
+				(font
+					(size 1.778 1.5113)
+				)
+				(justify left bottom)
+			)
+		)
+		(property "Footprint" "canGaugeDriver:DB9-MEAL"
+			(at 179.07 88.9 0)
+			(hide yes)
+			(show_name no)
+			(do_not_autoplace no)
+			(effects
+				(font
+					(size 1.27 1.27)
+				)
+			)
+		)
+		(property "Datasheet" ""
+			(at 179.07 88.9 0)
+			(hide yes)
+			(show_name no)
+			(do_not_autoplace no)
+			(effects
+				(font
+					(size 1.27 1.27)
+				)
+			)
+		)
+		(property "Description" ""
+			(at 179.07 88.9 0)
+			(hide yes)
+			(show_name no)
+			(do_not_autoplace no)
+			(effects
+				(font
+					(size 1.27 1.27)
+				)
+			)
+		)
+		(pin "3"
+		)
+		(pin "4"
+		)
+		(pin "7"
+		)
+		(pin "8"
+		)
+		(pin "2"
+		)
+		(pin "6"
+		)
+		(pin "1"
+		)
+		(pin "9"
+		)
+		(pin "5"
+		)
+		(instances
+			(project "canGaugeDriver"
+				(path "/53705195-86fb-46bf-a563-00a6cdeeae38"
+					(reference "J4")
+					(unit 1)
+				)
+			)
+		)
+	)
+	(symbol
 		(lib_id "Device:R_US")
 		(at 200.66 121.92 0)
@@
 	)
 	(symbol
-		(lib_id "power:GND")
-		(at 198.12 49.53 90)
-		(unit 1)
-		(body_style 1)
-		(exclude_from_sim no)
-		(in_bom yes)
-		(on_board yes)
-		(in_pos_files yes)
-		(dnp no)
-		(property "Reference" "#PWR09"
-			(at 204.47 49.53 0)
-			(hide yes)
-			(show_name no)
-			(do_not_autoplace no)
-			(effects
-				(font
-					(size 1.27 1.27)
-				)
-			)
-		)
-		(property "Value" "GND"
-			(at 200.66 48.514 90)
-			(show_name no)
-			(do_not_autoplace no)
-			(effects
-				(font
-					(size 1.27 1.27)
-				)
-				(justify right)
-			)
-		)
-		(property "Footprint" ""
-			(at 198.12 49.53 0)
-			(hide yes)
-			(show_name no)
-			(do_not_autoplace no)
-			(effects
-				(font
-					(size 1.27 1.27)
-				)
-			)
-		)
-		(property "Datasheet" ""
-			(at 198.12 49.53 0)
-			(hide yes)
-			(show_name no)
-			(do_not_autoplace no)
-			(effects
-				(font
-					(size 1.27 1.27)
-				)
-			)
-		)
-		(property "Description" "Power symbol creates a global label with name \"GND\" , ground"
-			(at 198.12 49.53 0)
-			(hide yes)
-			(show_name no)
-			(do_not_autoplace no)
-			(effects
-				(font
-					(size 1.27 1.27)
-				)
-			)
-		)
-		(pin "1"
-		)
-		(instances
-			(project "canGaugeDriver"
-				(path "/53705195-86fb-46bf-a563-00a6cdeeae38"
-					(reference "#PWR09")
-					(unit 1)
-				)
-			)
-		)
-	)
-	(symbol
 		(lib_id "Device:R_US")
 		(at 91.44 125.73 0)
@@
 	(symbol
 		(lib_id "power:GND")
+		(at 224.79 97.79 0)
+		(unit 1)
+		(body_style 1)
+		(exclude_from_sim no)
+		(in_bom yes)
+		(on_board yes)
+		(in_pos_files yes)
+		(dnp no)
+		(property "Reference" "#PWR09"
+			(at 224.79 104.14 0)
+			(hide yes)
+			(show_name no)
+			(do_not_autoplace no)
+			(effects
+				(font
+					(size 1.27 1.27)
+				)
+			)
+		)
+		(property "Value" "GND"
+			(at 225.806 100.33 0)
+			(hide yes)
+			(show_name no)
+			(do_not_autoplace no)
+			(effects
+				(font
+					(size 1.27 1.27)
+				)
+				(justify right)
+			)
+		)
+		(property "Footprint" ""
+			(at 224.79 97.79 0)
+			(hide yes)
+			(show_name no)
+			(do_not_autoplace no)
+			(effects
+				(font
+					(size 1.27 1.27)
+				)
+			)
+		)
+		(property "Datasheet" ""
+			(at 224.79 97.79 0)
+			(hide yes)
+			(show_name no)
+			(do_not_autoplace no)
+			(effects
+				(font
+					(size 1.27 1.27)
+				)
+			)
+		)
+		(property "Description" "Power symbol creates a global label with name \"GND\" , ground"
+			(at 224.79 97.79 0)
+			(hide yes)
+			(show_name no)
+			(do_not_autoplace no)
+			(effects
+				(font
+					(size 1.27 1.27)
+				)
+			)
+		)
+		(pin "1"
+		)
+		(instances
+			(project "canGaugeDriver"
+				(path "/53705195-86fb-46bf-a563-00a6cdeeae38"
+					(reference "#PWR09")
+					(unit 1)
+				)
+			)
+		)
+	)
+	(symbol
+		(lib_id "power:GND")
 		(at 43.18 185.42 0)
 		(unit 1)
@@
 			)
 		)
-		(property "Footprint" "CONN_SD-34826-001_24_MOL"
+		(property "Footprint" "MOLEX_348260240:CONN_SD-34826-001_24_MOL"
 			(at 228.6 38.1 0)
 			(hide yes)
